Commit message: feat(urdf): camera_optical_link — end-effector Arducam frame
Hand-authored fixed frame off gripper_frame_link for the claw-mounted Arducam
UC-844, so FK can walk straight to the camera instead of multiplying a Python
constant on afterwards. Identity rotation: the camera looks out along the claw's
reach and is not rolled, so the optical axes coincide with gripper_frame's.

Translation is CAD-derived, not hand-eye calibrated. x = 0.049413 = 0.02730
(claw underside, measured off wrist_roll_follower_so101_v1.stl: a flat face at
+27.30 mm spanning z = -95..-45) + 0.022113 (0.870604 in, sensor centre below
the hole centre). Camera hangs under the FIXED jaw; the moving jaw is on -x, so
the transform stays genuinely fixed rather than a function of gripper angle.

z = -0.0550 is provisional, scaled off a CAD screenshot and bounded to the flat
mounting face; it needs a real hole-centre measurement. A schematic 38 mm visual
box (visual only, no collision, so sim contact is unchanged) is offset -0.003113
in x so its top face lands flush on the claw underside without moving the optical
origin. Note the origin sits on the sensor centre, not the lens projection centre.

Marked as NOT generated by onshape-to-robot: re-exporting this URDF drops it.
camera.py's T_CAM_MOUNT still holds the superseded guess and is reconciled next.

Co-Authored-By: Claude Opus 5 <noreply@anthropic.com>

File: urdf/so101_new_calib.urdf (robot description, URDF)
Before this commit: robot so101_new_calib, 8 links, 7 joints
Links:
- added link camera_optical_link, mass 1e-9; visual box size=0.038 0.038 0.030
Joints:
- added joint camera_optical_joint: type fixed, parent gripper_frame_link, child camera_optical_link, origin xyz=0.049413 0 -0.0550 rpy=0 0 0, axis 0 0 0
